Commit message: fix(simulation): keep a single arm package

File: simulation/arm/urdf/so101_arm.urdf.xacro (robot description, xacro)
@@ -27,5 +27,5 @@
       <origin rpy="1.5707963 0 0" xyz="0 0.036394 -0.010422"/>
       <geometry>
-        <mesh filename="package://simulation/arm/meshes/body/part_001_Wiring_holder_v1.stl" scale="0.001 0.001 0.001"/>
+        <mesh filename="package://arm/meshes/body/part_001_Wiring_holder_v1.stl" scale="0.001 0.001 0.001"/>
       </geometry>
       <material name="so101_dark">
@@ -36,5 +36,5 @@
       <origin rpy="1.5707963 0 0" xyz="0 0.036394 -0.010422"/>
       <geometry>
-        <mesh filename="package://simulation/arm/meshes/body/part_001_Wiring_holder_v1.stl" scale="0.001 0.001 0.001"/>
+        <mesh filename="package://arm/meshes/body/part_001_Wiring_holder_v1.stl" scale="0.001 0.001 0.001"/>
       </geometry>
     </collision>
@@ -55,5 +55,5 @@
       <origin rpy="1.5707963 0 0" xyz="0 0 0"/>
       <geometry>
-        <mesh filename="package://simulation/arm/meshes/body/part_002_Wiring_holder_v1_1.stl" scale="0.001 0.001 0.001"/>
+        <mesh filename="package://arm/meshes/body/part_002_Wiring_holder_v1_1.stl" scale="0.001 0.001 0.001"/>
       </geometry>
       <material name="so101_dark">
@@ -65,5 +65,5 @@
       <origin rpy="1.5707963 0 0" xyz="0 0 0"/>
       <geometry>
-        <mesh filename="package://simulation/arm/meshes/body/part_086_1653192640.stl" scale="0.001 0.001 0.001"/>
+        <mesh filename="package://arm/meshes/body/part_086_1653192640.stl" scale="0.001 0.001 0.001"/>
       </geometry>
       <material name="servo_grey">
@@ -75,5 +75,5 @@
       <origin rpy="1.5707963 0 0" xyz="0 0 0"/>
       <geometry>
-        <mesh filename="package://simulation/arm/meshes/body/part_085_Extruded_1.stl" scale="0.001 0.001 0.001"/>
+        <mesh filename="package://arm/meshes/body/part_085_Extruded_1.stl" scale="0.001 0.001 0.001"/>
       </geometry>
       <material name="servo_grey">
@@ -84,5 +84,5 @@
       <origin rpy="1.5707963 0 0" xyz="0 0 0"/>
       <geometry>
-        <mesh filename="package://simulation/arm/meshes/body/part_002_Wiring_holder_v1_1.stl" scale="0.001 0.001 0.001"/>
+        <mesh filename="package://arm/meshes/body/part_002_Wiring_holder_v1_1.stl" scale="0.001 0.001 0.001"/>
       </geometry>
     </collision>
@@ -112,5 +112,5 @@
       <origin rpy="1.5707963 0 0" xyz="0.023656 0.119757 0.038947"/>
       <geometry>
-        <mesh filename="package://simulation/arm/meshes/body/part_003_Wiring_holder_v1_1.stl" scale="0.001 0.001 0.001"/>
+        <mesh filename="package://arm/meshes/body/part_003_Wiring_holder_v1_1.stl" scale="0.001 0.001 0.001"/>
       </geometry>
       <material name="so101_mid">
@@ -122,5 +122,5 @@
       <origin rpy="1.5707963 0 0" xyz="0.023656 0.119757 0.038947"/>
       <geometry>
-        <mesh filename="package://simulation/arm/meshes/body/part_087_736125216.stl" scale="0.001 0.001 0.001"/>
+        <mesh filename="package://arm/meshes/body/part_087_736125216.stl" scale="0.001 0.001 0.001"/>
       </geometry>
       <material name="servo_grey">
@@ -131,5 +131,5 @@
       <origin rpy="1.5707963 0 0" xyz="0.023656 0.119757 0.038947"/>
       <geometry>
-        <mesh filename="package://simulation/arm/meshes/body/part_003_Wiring_holder_v1_1.stl" scale="0.001 0.001 0.001"/>
+        <mesh filename="package://arm/meshes/body/part_003_Wiring_holder_v1_1.stl" scale="0.001 0.001 0.001"/>
       </geometry>
     </collision>
@@ -159,5 +159,5 @@
       <origin rpy="1.5707963 0 0" xyz="0.013895 0.148458 -0.073566"/>
       <geometry>
-        <mesh filename="package://simulation/arm/meshes/body/part_004_Wiring_holder_v1_2.stl" scale="0.001 0.001 0.001"/>
+        <mesh filename="package://arm/meshes/body/part_004_Wiring_holder_v1_2.stl" scale="0.001 0.001 0.001"/>
       </geometry>
       <material name="so101_light">
@@ -169,5 +169,5 @@
       <origin rpy="1.5707963 0 0" xyz="0.013895 0.148458 -0.073566"/>
       <geometry>
-        <mesh filename="package://simulation/arm/meshes/body/part_088_1653192640_1.stl" scale="0.001 0.001 0.001"/>
+        <mesh filename="package://arm/meshes/body/part_088_1653192640_1.stl" scale="0.001 0.001 0.001"/>
       </geometry>
       <material name="servo_grey">
@@ -178,5 +178,5 @@
       <origin rpy="1.5707963 0 0" xyz="0.013895 0.148458 -0.073566"/>
       <geometry>
-        <mesh filename="package://simulation/arm/meshes/body/part_004_Wiring_holder_v1_2.stl" scale="0.001 0.001 0.001"/>
+        <mesh filename="package://arm/meshes/body/part_004_Wiring_holder_v1_2.stl" scale="0.001 0.001 0.001"/>
       </geometry>
     </collision>
@@ -206,5 +206,5 @@
       <origin rpy="1.5707963 0 0" xyz="-0.005534 0.152613 0.060418"/>
       <geometry>
-        <mesh filename="package://simulation/arm/meshes/body/part_008_Wiring_holder_v1_1__2.stl" scale="0.001 0.001 0.001"/>
+        <mesh filename="package://arm/meshes/body/part_008_Wiring_holder_v1_1__2.stl" scale="0.001 0.001 0.001"/>
       </geometry>
       <material name="so101_light">
@@ -216,5 +216,5 @@
       <origin rpy="1.5707963 0 0" xyz="-0.005534 0.152613 0.060418"/>
       <geometry>
-        <mesh filename="package://simulation/arm/meshes/body/part_089_1653192640_2.stl" scale="0.001 0.001 0.001"/>
+        <mesh filename="package://arm/meshes/body/part_089_1653192640_2.stl" scale="0.001 0.001 0.001"/>
       </geometry>
       <material name="servo_grey">
@@ -225,5 +225,5 @@
       <origin rpy="1.5707963 0 0" xyz="-0.005534 0.152613 0.060418"/>
       <geometry>
-        <mesh filename="package://simulation/arm/meshes/body/part_008_Wiring_holder_v1_1__2.stl" scale="0.001 0.001 0.001"/>
+        <mesh filename="package://arm/meshes/body/part_008_Wiring_holder_v1_1__2.stl" scale="0.001 0.001 0.001"/>
       </geometry>
     </collision>
@@ -260,5 +260,5 @@
       <origin rpy="0 0 1.5707963" xyz="0 0 0"/>
       <geometry>
-        <mesh filename="package://simulation/arm/meshes/end_effector/part_002_solid_002.stl" scale="0.001 0.001 0.001"/>
+        <mesh filename="package://arm/meshes/end_effector/part_002_solid_002.stl" scale="0.001 0.001 0.001"/>
       </geometry>
       <material name="gripper_dark">
@@ -269,5 +269,5 @@
       <origin rpy="0 0 1.5707963" xyz="0 0 0"/>
       <geometry>
-        <mesh filename="package://simulation/arm/meshes/end_effector/part_001_solid_001.stl" scale="0.001 0.001 0.001"/>
+        <mesh filename="package://arm/meshes/end_effector/part_001_solid_001.stl" scale="0.001 0.001 0.001"/>
       </geometry>
       <material name="gripper_light">
@@ -278,5 +278,5 @@
       <origin rpy="0 0 1.5707963" xyz="0 0 0"/>
       <geometry>
-        <mesh filename="package://simulation/arm/meshes/end_effector/part_002_solid_002.stl" scale="0.001 0.001 0.001"/>
+        <mesh filename="package://arm/meshes/end_effector/part_002_solid_002.stl" scale="0.001 0.001 0.001"/>
       </geometry>
     </collision>

File: simulation/arm/urdf/so101_arm_camera.urdf.xacro (robot description, xacro)
@@ -27,5 +27,5 @@
       <origin rpy="1.5707963 0 0" xyz="0 0.036394 -0.010422"/>
       <geometry>
-        <mesh filename="package://simulation/arm/meshes/body/part_001_Wiring_holder_v1.stl" scale="0.001 0.001 0.001"/>
+        <mesh filename="package://arm/meshes/body/part_001_Wiring_holder_v1.stl" scale="0.001 0.001 0.001"/>
       </geometry>
       <material name="so101_dark">
@@ -36,5 +36,5 @@
       <origin rpy="1.5707963 0 0" xyz="0 0.036394 -0.010422"/>
       <geometry>
-        <mesh filename="package://simulation/arm/meshes/body/part_001_Wiring_holder_v1.stl" scale="0.001 0.001 0.001"/>
+        <mesh filename="package://arm/meshes/body/part_001_Wiring_holder_v1.stl" scale="0.001 0.001 0.001"/>
       </geometry>
     </collision>
@@ -55,5 +55,5 @@
       <origin rpy="1.5707963 0 0" xyz="0 0 0"/>
       <geometry>
-        <mesh filename="package://simulation/arm/meshes/body/part_002_Wiring_holder_v1_1.stl" scale="0.001 0.001 0.001"/>
+        <mesh filename="package://arm/meshes/body/part_002_Wiring_holder_v1_1.stl" scale="0.001 0.001 0.001"/>
       </geometry>
       <material name="so101_dark">
@@ -65,5 +65,5 @@
       <origin rpy="1.5707963 0 0" xyz="0 0 0"/>
       <geometry>
-        <mesh filename="package://simulation/arm/meshes/body/part_086_1653192640.stl" scale="0.001 0.001 0.001"/>
+        <mesh filename="package://arm/meshes/body/part_086_1653192640.stl" scale="0.001 0.001 0.001"/>
       </geometry>
       <material name="servo_grey">
@@ -75,5 +75,5 @@
       <origin rpy="1.5707963 0 0" xyz="0 0 0"/>
       <geometry>
-        <mesh filename="package://simulation/arm/meshes/body/part_085_Extruded_1.stl" scale="0.001 0.001 0.001"/>
+        <mesh filename="package://arm/meshes/body/part_085_Extruded_1.stl" scale="0.001 0.001 0.001"/>
       </geometry>
       <material name="servo_grey">
@@ -84,5 +84,5 @@
       <origin rpy="1.5707963 0 0" xyz="0 0 0"/>
       <geometry>
-        <mesh filename="package://simulation/arm/meshes/body/part_002_Wiring_holder_v1_1.stl" scale="0.001 0.001 0.001"/>
+        <mesh filename="package://arm/meshes/body/part_002_Wiring_holder_v1_1.stl" scale="0.001 0.001 0.001"/>
       </geometry>
     </collision>
@@ -112,5 +112,5 @@
       <origin rpy="1.5707963 0 0" xyz="0.023656 0.119757 0.038947"/>
       <geometry>
-        <mesh filename="package://simulation/arm/meshes/body/part_003_Wiring_holder_v1_1.stl" scale="0.001 0.001 0.001"/>
+        <mesh filename="package://arm/meshes/body/part_003_Wiring_holder_v1_1.stl" scale="0.001 0.001 0.001"/>
       </geometry>
       <material name="so101_mid">
@@ -122,5 +122,5 @@
       <origin rpy="1.5707963 0 0" xyz="0.023656 0.119757 0.038947"/>
       <geometry>
-        <mesh filename="package://simulation/arm/meshes/body/part_087_736125216.stl" scale="0.001 0.001 0.001"/>
+        <mesh filename="package://arm/meshes/body/part_087_736125216.stl" scale="0.001 0.001 0.001"/>
       </geometry>
       <material name="servo_grey">
@@ -131,5 +131,5 @@
       <origin rpy="1.5707963 0 0" xyz="0.023656 0.119757 0.038947"/>
       <geometry>
-        <mesh filename="package://simulation/arm/meshes/body/part_003_Wiring_holder_v1_1.stl" scale="0.001 0.001 0.001"/>
+        <mesh filename="package://arm/meshes/body/part_003_Wiring_holder_v1_1.stl" scale="0.001 0.001 0.001"/>
       </geometry>
     </collision>
@@ -159,5 +159,5 @@
       <origin rpy="1.5707963 0 0" xyz="0.013895 0.148458 -0.073566"/>
       <geometry>
-        <mesh filename="package://simulation/arm/meshes/body/part_004_Wiring_holder_v1_2.stl" scale="0.001 0.001 0.001"/>
+        <mesh filename="package://arm/meshes/body/part_004_Wiring_holder_v1_2.stl" scale="0.001 0.001 0.001"/>
       </geometry>
       <material name="so101_light">
@@ -169,5 +169,5 @@
       <origin rpy="1.5707963 0 0" xyz="0.013895 0.148458 -0.073566"/>
       <geometry>
-        <mesh filename="package://simulation/arm/meshes/body/part_088_1653192640_1.stl" scale="0.001 0.001 0.001"/>
+        <mesh filename="package://arm/meshes/body/part_088_1653192640_1.stl" scale="0.001 0.001 0.001"/>
       </geometry>
       <material name="servo_grey">
@@ -178,5 +178,5 @@
       <origin rpy="1.5707963 0 0" xyz="0.013895 0.148458 -0.073566"/>
       <geometry>
-        <mesh filename="package://simulation/arm/meshes/body/part_004_Wiring_holder_v1_2.stl" scale="0.001 0.001 0.001"/>
+        <mesh filename="package://arm/meshes/body/part_004_Wiring_holder_v1_2.stl" scale="0.001 0.001 0.001"/>
       </geometry>
     </collision>
@@ -206,5 +206,5 @@
       <origin rpy="1.5707963 0 0" xyz="-0.005534 0.152613 0.060418"/>
       <geometry>
-        <mesh filename="package://simulation/arm/meshes/body/part_008_Wiring_holder_v1_1__2.stl" scale="0.001 0.001 0.001"/>
+        <mesh filename="package://arm/meshes/body/part_008_Wiring_holder_v1_1__2.stl" scale="0.001 0.001 0.001"/>
       </geometry>
       <material name="so101_light">
@@ -216,5 +216,5 @@
       <origin rpy="1.5707963 0 0" xyz="-0.005534 0.152613 0.060418"/>
       <geometry>
-        <mesh filename="package://simulation/arm/meshes/body/part_089_1653192640_2.stl" scale="0.001 0.001 0.001"/>
+        <mesh filename="package://arm/meshes/body/part_089_1653192640_2.stl" scale="0.001 0.001 0.001"/>
       </geometry>
       <material name="servo_grey">
@@ -225,5 +225,5 @@
       <origin rpy="1.5707963 0 0" xyz="-0.005534 0.152613 0.060418"/>
       <geometry>
-        <mesh filename="package://simulation/arm/meshes/body/part_008_Wiring_holder_v1_1__2.stl" scale="0.001 0.001 0.001"/>
+        <mesh filename="package://arm/meshes/body/part_008_Wiring_holder_v1_1__2.stl" scale="0.001 0.001 0.001"/>
       </geometry>
     </collision>
@@ -260,5 +260,5 @@
       <origin rpy="0 0 1.5707963" xyz="0 0 0"/>
       <geometry>
-        <mesh filename="package://simulation/arm/meshes/end_effector/part_002_solid_002.stl" scale="0.001 0.001 0.001"/>
+        <mesh filename="package://arm/meshes/end_effector/part_002_solid_002.stl" scale="0.001 0.001 0.001"/>
       </geometry>
       <material name="gripper_dark">
@@ -269,5 +269,5 @@
       <origin rpy="0 0 1.5707963" xyz="0 0 0"/>
       <geometry>
-        <mesh filename="package://simulation/arm/meshes/end_effector/part_001_solid_001.stl" scale="0.001 0.001 0.001"/>
+        <mesh filename="package://arm/meshes/end_effector/part_001_solid_001.stl" scale="0.001 0.001 0.001"/>
       </geometry>
       <material name="gripper_light">
@@ -278,5 +278,5 @@
       <origin rpy="0 0 1.5707963" xyz="0 0 0"/>
       <geometry>
-        <mesh filename="package://simulation/arm/meshes/end_effector/part_002_solid_002.stl" scale="0.001 0.001 0.001"/>
+        <mesh filename="package://arm/meshes/end_effector/part_002_solid_002.stl" scale="0.001 0.001 0.001"/>
       </geometry>
     </collision>
@@ -322,5 +322,5 @@
       <origin rpy="1.5707963 0 0" xyz="0.060129397 -0.021552011 0.011971371"/>
       <geometry>
-        <mesh filename="package://simulation/arm/meshes/cam_holder/part_003_surface_shell_003.stl" scale="0.001 0.001 0.001"/>
+        <mesh filename="package://arm/meshes/cam_holder/part_003_surface_shell_003.stl" scale="0.001 0.001 0.001"/>
       </geometry>
       <material name="camera_holder_black">
@@ -331,5 +331,5 @@
       <origin rpy="1.5707963 0 0" xyz="0.060129397 -0.021552011 0.011971371"/>
       <geometry>
-        <mesh filename="package://simulation/arm/meshes/cam_holder/part_003_surface_shell_003.stl" scale="0.001 0.001 0.001"/>
+        <mesh filename="package://arm/meshes/cam_holder/part_003_surface_shell_003.stl" scale="0.001 0.001 0.001"/>
       </geometry>
     </collision>
