Commit message: feat(control): deliver SO-101 real-arm runtime

File: simulation/so-101_description/urdf/so101_arm_macro.urdf.xacro (robot description, xacro)
@@ -139,5 +139,5 @@
       <child link="${prefix}arm_upper"/>
       <axis xyz="0.99996 -0.000076 0.008726"/>
-      <limit lower="-1.57" upper="1.57" effort="10" velocity="5"/>
+      <limit lower="-0.5236" upper="2.9" effort="10" velocity="5"/>
       <dynamics damping="0.1"/>
     </joint>
@@ -177,5 +177,5 @@
       <child link="${prefix}arm_lower"/>
       <axis xyz="-0.99992 0.008802 -0.008650"/>
-      <limit lower="-1.57" upper="1.57" effort="10" velocity="5"/>
+      <limit lower="0" upper="3.14" effort="10" velocity="5"/>
       <dynamics damping="0.1"/>
     </joint>
@@ -260,5 +260,5 @@
       <child link="${prefix}gripper_base"/>
       <axis xyz="0 0 1"/>
-      <limit lower="-1.57" upper="1.57" effort="10" velocity="5"/>
+      <limit lower="-3.14" upper="3.14" effort="10" velocity="5"/>
       <dynamics damping="0.1"/>
     </joint>
